Commit message: Have local costmap and lidar adjustments

File: diff_drive_edubot/config/diff_drive_gazebo.xacro (robot description, xacro)
@@ -8,4 +8,8 @@
         <parameters>$(find diff_drive)/config/ros2_controllers.yaml</parameters>
         <parameters>$(find diff_drive)/config/gz_use_sim.yaml</parameters>
+        <ros>
+          <remapping>/diffbot_base_controller/cmd_vel_unstamped:=/cmd_vel</remapping>
+          <remapping>/diffbot_base_controller/odom:=/odom</remapping>
+        </ros>
       </plugin>
     </gazebo>

File: diff_drive_edubot/config/lidar.xacro (robot description, xacro)
@@ -2,10 +2,11 @@
 <robot xmlns:xacro="http://www.ros.org/wiki/xacro" >
     <joint name="laser_joint" type="fixed">
-        <parent link="chassis"/>
+        <parent link="base_link"/>
         <child link="laser_frame"/>
-        <origin xyz="0.122 0 0.212" rpy="0 0 0"/>
+        <origin xyz="0.085 0 0.08" rpy="0 0 0"/>
     </joint>
     <link name="laser_frame">
         <visual>
+            <origin xyz="0 0 -0.05"/>
             <geometry>
                 <cylinder radius="0.05" length="0.04"/>
@@ -32,23 +33,31 @@
         <material>Gazebo/Black</material>
         <sensor name="laser" type="ray">
-            <pose> 0 0 0 0 0 0 </pose>
+            <always_on>true</always_on>
             <visualize>true</visualize>
-            <update_rate>10</update_rate>
+            <pose>-0.064 0 0.121 0 0 0</pose>
+            <update_rate>5</update_rate>
             <ray>
-                <scan>
-                    <horizontal>
-                        <samples>360</samples>
-                        <min_angle>-3.14</min_angle>
-                        <max_angle>3.14</max_angle>
-                    </horizontal>
-                </scan>
-                <range>
-                    <min>0.3</min>
-                    <max>12</max>
-                </range>
+            <scan>
+                <horizontal>
+                <samples>599.6944232238</samples> <!-- 599.6944232238 -->
+                <resolution>1.000000</resolution>
+                <min_angle>4.97419</min_angle>
+                <max_angle>7.59218</max_angle>
+                </horizontal>
+            </scan>
+            <range>
+                <min>0.120000</min>
+                <max>3.5</max>
+                <resolution>0.015000</resolution>
+            </range>
+            <noise>
+                <type>gaussian</type>
+                <mean>0.0</mean>
+                <stddev>0.01</stddev>
+            </noise>
             </ray>
             <plugin name="laser_controller" filename="libgazebo_ros_ray_sensor.so">
                 <ros>
-                    <argument>~/out:=scan</argument>
+                    <remapping>~/out:=scan</remapping>
                 </ros>
                 <output_type>sensor_msgs/LaserScan</output_type>
