Commit message: Project almost completed

File: pattern_matcher/urdf/pattern.urdf (robot description, URDF)
Before this commit: robot pattern, 2 links, 1 joints
Links:
- link pattern_mesh: geometry collision mesh filename=$(find pattern_matcher)/meshes/pattern.STL scale=0.001 0.001 0.001; visual mesh filename=$(find pattern_matcher)/meshes/pattern.STL scale=0.001 0.001 0.001

Commit message: Added files for new doching system

File: pattern_matcher/urdf/pattern.urdf (robot description, URDF)
Before this commit: robot pattern, 2 links, 1 joints
Links:
- link pattern_mesh: geometry collision mesh filename=$(find pattern_matcher)/meshes/docking_education_robot.STL scale=0.001 0.001 0.001; visual mesh filename=$(find pattern_matcher)/meshes/docking_education_robot.STL scale=0.001 0.001 0.001

Commit message: Minute fix to urd of pattern mesh

File: pattern_matcher/urdf/pattern.urdf (robot description, URDF)
Before this commit: robot pattern, 2 links, 1 joints
Links:
- removed link world
- added link map
Joints:
- joint pattern_joint: parent world -> map
